File: main.brd (EAGLE design)
At the start: 53.3 x 68.6 mm, 33 parts, among them IC1 4050D, U1 MCP2551, U2 STN1110

Commit message: Review phase 1
Parts:
- added R13: 100k, resistor:0204/7
- U2: value STN1110 -> STN1100
Connections:
- net 3.3V: now also R13.1
- net GND: now also U2.11; no longer U2.7
- net ~OBD_TX_LED/~RST_NVM: now also R13.2
Routing:
- net GND: track 262.5 -> 259.2 mm
- net 3.3V: track 155.2 -> 158.4 mm
- net ~OBD_TX_LED/~RST_NVM: track 4.52 -> 7.65 mm
Changed lines of the file:
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@@
 <attribute name="VALUE" x="8.278" y="56.667" size="1.27" layer="27" ratio="10" rot="R180"/>
 </element>
-<element name="U2" library="personal" package="SOCKET-28-3" value="STN1110" x="27" y="21" smashed="yes" rot="R270">
+<element name="U2" library="personal" package="SOCKET-28-3" value="STN1100" x="27" y="21" smashed="yes" rot="R270">
 <attribute name="VALUE" x="26.565" y="24.109" size="1.27" layer="25" ratio="10" rot="R270"/>
 </element>
@@
 </element>
 <element name="R9" library="resistor" package="0204/7" value="330" x="38" y="26"/>
-<element name="R10" library="resistor" package="0204/7" value="330" x="38" y="20"/>
+<element name="R10" library="resistor" package="0204/7" value="330" x="38" y="20" smashed="yes">
+<attribute name="NAME" x="35.46" y="21.2954" size="0.9906" layer="25" ratio="10"/>
+<attribute name="VALUE" x="36.3744" y="19.5174" size="0.9906" layer="27" ratio="10"/>
+</element>
 <element name="LED1" library="led" package="DUOLED-A-3MM" value="OBD RX/TX" x="45" y="23" smashed="yes" rot="R270">
 <attribute name="VALUE" x="46.96" y="27.69" size="1.27" layer="25" ratio="10" rot="R270"/>
@@
 </element>
 <element name="U$2" library="SparkFun-Aesthetics" package="OSHW-LOGO-S" value="" x="7.62" y="1.905"/>
+<element name="R13" library="resistor" package="0204/7" value="100k" x="38.1" y="22.86" smashed="yes" rot="R180">
+<attribute name="NAME" x="38.1" y="24.7396" size="0.9906" layer="25" ratio="10" rot="R180"/>
+<attribute name="VALUE" x="39.7256" y="23.3426" size="0.9906" layer="27" ratio="10" rot="R180"/>
+</element>
 </elements>
 <signals>
@@
 <contactref element="U2" pad="5"/>
 <contactref element="U2" pad="8"/>
-<contactref element="U2" pad="7"/>
 <contactref element="R12" pad="1"/>
 <contactref element="JP1" pad="1"/>
 <contactref element="ARDUINO1" pad="GND2"/>
 <contactref element="ARDUINO1" pad="GND3"/>
-<wire x1="23.94" y1="21.86" x2="23.94" y2="19.32" width="0.254" layer="1"/>
-<wire x1="23.94" y1="19.32" x2="23.19" y2="19.73" width="0.254" layer="1"/>
-<wire x1="23.94" y1="21.86" x2="23.19" y2="22.27" width="0.254" layer="1"/>
 <wire x1="35.37" y1="14.24" x2="31.56" y2="14.24" width="0.254" layer="1"/>
 <wire x1="31.56" y1="14.24" x2="30.81" y2="14.65" width="0.254" layer="1"/>
 <wire x1="35.37" y1="14.24" x2="35.56" y2="14.7" width="0.254" layer="1"/>
-<wire x1="29.02" y1="14.24" x2="23.94" y2="19.32" width="0.254" layer="16"/>
+<wire x1="29.02" y1="14.24" x2="25.4" y2="17.78" width="0.254" layer="16"/>
+<wire x1="25.4" y1="17.78" x2="23.94" y2="19.32" width="0.254" layer="16"/>
 <wire x1="30.29" y1="14.24" x2="29.02" y2="14.24" width="0.254" layer="16"/>
 <wire x1="23.94" y1="19.32" x2="23.19" y2="19.73" width="0.254" layer="16"/>
@@
 <wire x1="2.35" y1="21.86" x2="2.14" y2="22" width="0.254" layer="1"/>
 <wire x1="2.35" y1="24.4" x2="2.14" y2="24.54" width="0.254" layer="1"/>
-<wire x1="2.35" y1="21.86" x2="7.53" y2="21.88" width="0.254" layer="16"/>
-<wire x1="7.53" y1="21.88" x2="7.9" y2="21.88" width="0.254" layer="16"/>
-<wire x1="7.9" y1="21.88" x2="7.9" y2="11.8" width="0.254" layer="16"/>
-<wire x1="7.9" y1="11.8" x2="12.51" y2="11.7" width="0.254" layer="16"/>
-<wire x1="12.51" y1="11.7" x2="12.43" y2="11.43" width="0.254" layer="16"/>
-<wire x1="2.35" y1="21.86" x2="2.14" y2="22" width="0.254" layer="16"/>
-<wire x1="7.53" y1="21.88" x2="12.51" y2="21.86" width="0.254" layer="16"/>
-<wire x1="12.51" y1="21.86" x2="12.43" y2="21.59" width="0.254" layer="16"/>
-<wire x1="12.51" y1="23.13" x2="18.86" y2="29.48" width="0.254" layer="1"/>
-<wire x1="12.51" y1="21.86" x2="12.51" y2="23.13" width="0.254" layer="1"/>
-<wire x1="18.86" y1="29.48" x2="19" y2="29.73" width="0.254" layer="1"/>
-<wire x1="12.51" y1="21.86" x2="22.67" y2="21.86" width="0.254" layer="1"/>
-<wire x1="22.67" y1="21.86" x2="23.19" y2="22.27" width="0.254" layer="1"/>
-<wire x1="12.51" y1="21.86" x2="12.43" y2="21.59" width="0.254" layer="1"/>
 <wire x1="6.76" y1="54.01" x2="6.76" y2="50" width="0.254" layer="1"/>
 <wire x1="6.76" y1="54.01" x2="7.23" y2="54" width="0.254" layer="1"/>
@@
 <wire x1="37.084" y1="56.134" x2="36.23" y2="56.93" width="0.1524" layer="1"/>
 <wire x1="38.354" y1="51.816" x2="38.555" y2="51.6734" width="0.1524" layer="1"/>
+<wire x1="11.176" y1="12.446" x2="12.192" y2="11.43" width="0.1524" layer="1"/>
+<wire x1="11.176" y1="20.574" x2="11.176" y2="12.446" width="0.1524" layer="1"/>
+<wire x1="12.192" y1="21.59" x2="11.176" y2="20.574" width="0.1524" layer="1"/>
+<wire x1="12.192" y1="11.43" x2="12.43" y2="11.43" width="0.1524" layer="1"/>
+<wire x1="12.192" y1="21.59" x2="12.43" y2="21.59" width="0.1524" layer="1"/>
+<wire x1="2.54" y1="21.59" x2="2.286" y2="21.844" width="0.1524" layer="16"/>
+<wire x1="12.43" y1="21.59" x2="2.54" y2="21.59" width="0.1524" layer="16"/>
+<wire x1="2.286" y1="21.844" x2="2.14" y2="22" width="0.1524" layer="16"/>
+<wire x1="18.796" y1="27.94" x2="17.018" y2="26.162" width="0.1524" layer="1"/>
+<wire x1="17.018" y1="26.162" x2="12.446" y2="21.59" width="0.1524" layer="1"/>
+<wire x1="18.796" y1="29.718" x2="18.796" y2="27.94" width="0.1524" layer="1"/>
+<wire x1="12.446" y1="21.59" x2="12.43" y2="21.59" width="0.1524" layer="1"/>
+<wire x1="18.796" y1="29.718" x2="19" y2="29.73" width="0.1524" layer="1"/>
+<wire x1="17.018" y1="25.908" x2="23.114" y2="19.812" width="0.1524" layer="1"/>
+<wire x1="17.018" y1="26.162" x2="17.018" y2="25.908" width="0.1524" layer="1"/>
+<wire x1="23.114" y1="19.812" x2="23.19" y2="19.73" width="0.1524" layer="1"/>
+<contactref element="U2" pad="11"/>
+<wire x1="25.4" y1="17.78" x2="25.4" y2="13.97" width="0.1524" layer="16"/>
+<wire x1="25.4" y1="13.97" x2="23.368" y2="12.192" width="0.1524" layer="16"/>
+<wire x1="23.368" y1="12.192" x2="23.19" y2="12.11" width="0.1524" layer="16"/>
 </signal>
 <signal name="N$3">
@@
 <via x="43.942" y="57.912" extent="1-16" drill="0.3048"/>
 <via x="46.99" y="54.864" extent="1-16" drill="0.3048"/>
+<contactref element="R13" pad="1"/>
+<wire x1="44.958" y1="22.86" x2="41.91" y2="22.86" width="0.1524" layer="1"/>
+<wire x1="44.958" y1="22.86" x2="45" y2="23" width="0.1524" layer="1"/>
 </signal>
 <signal name="CAN_TX">
@@
 <wire x1="31.56" y1="19.32" x2="30.81" y2="19.73" width="0.254" layer="16"/>
 <wire x1="34.1" y1="20.59" x2="34.19" y2="20" width="0.254" layer="16"/>
+<contactref element="R13" pad="2"/>
+<wire x1="34.29" y1="20.574" x2="34.29" y2="22.86" width="0.1524" layer="16"/>
+<wire x1="34.036" y1="20.574" x2="34.29" y2="20.574" width="0.1524" layer="16"/>
+<wire x1="34.036" y1="20.574" x2="34.19" y2="20" width="0.1524" layer="16"/>
 </signal>
 <signal name="~OBD_RX_LED/INT">

Commit message: Ready to print\!
Parts:
- added C9: 1uF, capacitor-wima:C2.5-2
- added SW_SERIAL: M02LOCK, SparkFun-Connectors:1X02_LOCK
- moved JP1 5.39 mm to (39.2, 12.2), turned to 0 degrees
Connections:
- new net SLEEP: ARDUINO1.02, U2.12
- net 3.3V: now also C9.1
- net GND: now also C9.2
- net GPS_RX: now also SW_SERIAL.2; no longer ARDUINO1.05
- net GPS_TX: now also SW_SERIAL.1; no longer ARDUINO1.06
Routing:
- net SLEEP: track 0.00 -> 36.1 mm
- net GND: track 259.2 -> 263.6 mm
- net UART_RX: track 23.7 -> 21.9 mm, vias 0 -> 1
- net GPS_RX: track 8.88 -> 10.5 mm
- net GPS_TX: track 8.96 -> 10.4 mm
